Commit message: descripcion de los cambios

File: src/scara_description/urdf/scara.urdf.xacro (robot description, xacro)
@@ -76,5 +76,5 @@
     <parent link="link_2"/>
     <child link="link_p"/>
-    <origin xyz="${l2} 0 ${h3}"/>
+    <origin xyz="${l2} 0.001 ${h3}"/>
     <axis xyz="0 0 -1"/>
     <limit lower="0.0" upper="${p_max}" effort="50" velocity="0.01"/>
